Commit message: minor changes

File: robosense_description/urdf/RS-16.urdf.xacro (robot description, xacro)
@@ -57,5 +57,6 @@
               </horizontal>
               <vertical>
-                <samples>${lasers}</samples>
+                <!-- <samples>${lasers}</samples> -->
+                <samples>64</samples>
                 <resolution>1</resolution>
                 <min_angle>-${15.0*M_PI/180.0}</min_angle>
@@ -76,5 +77,5 @@
           <plugin name="gazebo_ros_laser_controller" filename="libgazebo_ros_robosense_gpu_laser.so">
             <topicName>${topic}</topicName>
-            <frameName>${name}</frameName>
+            <frameName>/${name}_base_link</frameName>
             <min_range>${min_range}</min_range>
             <max_range>${max_range}</max_range>
@@ -116,5 +117,5 @@
           <plugin name="gazebo_ros_laser_controller" filename="libgazebo_ros_robosense_laser.so">
             <topicName>${topic}</topicName>
-            <frameName>${name}</frameName>
+            <frameName>/${name}_base_link</frameName>
             <min_range>${min_range}</min_range>
             <max_range>${max_range}</max_range>

File: robosense_description/urdf/example.urdf.xacro (robot description, xacro)
@@ -3,13 +3,26 @@
   <xacro:arg name="gpu" default="false"/>
   <xacro:property name="gpu" value="$(arg gpu)" />
+  <xacro:arg name="ns" default="sensor0"/>
+  <xacro:property name="ns" value="$(arg ns)" />
+  <xacro:arg name="x" default="0.0"/>
+  <xacro:arg name="y" default="0.0"/>
+  <xacro:property name="x" value="$(arg x)" />
+  <xacro:property name="y" value="$(arg y)" />
   <!-- Base Footprint -->
-  <link name="base_footprint" />
+  <link name="${ns}_mount_base_footprint">
+      <!-- <visual>
+          <origin xyz="${x} ${y} 0.05" rpy="0 0 0" />
+      </visual>
+      <collision>
+          <origin xyz="${x} ${y} 0.05" rpy="0 0 0" />
+      </collision> -->
+  </link>
   <!-- Base Link -->
   <joint name="footprint" type="fixed" >
-   <parent link="base_footprint" />
-    <child link="base_link" />
+    <parent link="${ns}_mount_base_footprint" />
+    <child link="${ns}_mount_base_link" />
     <origin xyz="0 0 0.05" rpy="0 0 0" />
   </joint>
-  <link name="base_link" >
+  <link name="${ns}_mount_base_link" >
     <visual>
       <geometry>
@@ -31,5 +44,5 @@
   </link>
   <xacro:include filename="$(find robosense_description)/urdf/RS-16.urdf.xacro"/>
-  <RS-16 parent="base_link" name="robosense" topic="/rs_points" hz="20" samples="900" gpu="${gpu}">
+  <RS-16 parent="${ns}_mount_base_link" name="${ns}" topic="/${ns}/rs_points" hz="20" samples="900" gpu="${gpu}">
     <origin xyz="0 0 0.4" rpy="0 0 0" />
   </RS-16>
